File: Hardware/KiCAD/Meanwell IRM Board.kicad_pcb (KiCad board)
At the start: 2 copper layers, 88.3 x 85.2 mm, 12 parts, among them J1 AC/L, J2 AC/N, J3 V-Combine, J4 V1, J5 V2

Commit message: started doing todos
Parts:
- added D1: LED_gr, LED_SMD:LED_0805_2012Metric_Pad1.15x1.40mm_HandSolder, F.Cu at (214.7, 100.2)
- added D2: LED_gr, LED_SMD:LED_0805_2012Metric_Pad1.15x1.40mm_HandSolder, F.Cu at (214.7, 103.2)
- added J6: Dual_Out, Connector_JST:JST_XH_B4B-XH-A_1x04_P2.50mm_Vertical, F.Cu at (194.2, 107.4)
- added R1: 10k, Resistor_SMD:R_0805_2012Metric_Pad1.20x1.40mm_HandSolder, F.Cu at (219.4, 100.2)
- added R2: 10k, Resistor_SMD:R_0805_2012Metric_Pad1.20x1.40mm_HandSolder, F.Cu at (219.4, 103.1)
- J4, J5: footprint Connector_JST:JST_EH_B2B-EH-A_1x02_P2.50mm_Vertical -> Connector_JST:JST_XH_B2B-XH-A_1x02_P2.50mm_Vertical
- moved H4 16.2 mm to (104.8, 143.4)
- moved H3 16.2 mm to (185.5, 143.4)
- moved J3 16.2 mm to (183.8, 104.0)
- moved PS1 16.2 mm to (137.1, 80.7)
- moved PS2 16.2 mm to (137.1, 121.0)
- moved H1 16.2 mm to (104.8, 65.8)
- moved J1 16.2 mm to (108.8, 83.1)
- moved J2 16.2 mm to (108.8, 98.0)
- moved J4 16.2 mm to (184.2, 81.3)
- moved G*** 16.2 mm to (143.2, 104.0)
- moved H2 16.2 mm to (185.5, 65.8)
- moved J5 16.1 mm to (183.7, 126.2)
Connections:
- net Net-(J3-Pin_1) renamed VSS_A
- net Net-(J3-Pin_2) renamed VDD_B
- net Net-(J4-Pin_1) renamed VDD_A
- net Net-(J5-Pin_2) renamed VSS_B
Other:
- board size 88.3 x 85.2 mm -> 100 x 85.2 mm
