File: Hardware/KiCAD/Meanwell IRM Board.kicad_sch (KiCad schematic)
At the start: 11 parts, among them J1 AC/L, J2 AC/N, J3 V-Combine, J4 V1, J5 V2

Commit message: added reichelt nr for connectors
Parts:
- J1, J2: Reichelt Nr. (none) -> VT FS-P 4,75
Changed lines of the file:
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@@
+			)
+		)
+		(property "Reichelt Nr." "VT FS-P 4,75"
+			(at 71.12 41.275 0)
+			(effects
+				(font
+					(size 1.27 1.27)
+				)
 			)
 		)
@@
 			)
 		)
-		(property "Reichelt Nr." ""
-			(at 71.12 36.195 0)
-			(effects
+		(property "Reichelt Nr." "VT FS-P 4,75"
+			(at 71.12 36.195 0)
+			(effects

Commit message: started doing todos
Parts:
- added D1, D2: LED_gr, LED_SMD:LED_0805_2012Metric_Pad1.15x1.40mm_HandSolder, symbol Device:LED_Small
- added J6: Dual_Out, Connector_JST:JST_XH_B4B-XH-A_1x04_P2.50mm_Vertical, symbol Connector:Conn_01x04_Socket
- added R1, R2: 10k, Resistor_SMD:R_0805_2012Metric_Pad1.20x1.40mm_HandSolder, symbol Device:R_Small
- J4, J5: footprint Connector_JST:JST_EH_B2B-EH-A_1x02_P2.50mm_Vertical -> Connector_JST:JST_XH_B2B-XH-A_1x02_P2.50mm_Vertical
Connections:
- net VDD_A: now reaches J4.1 (Pin_1), PS1.4 (+Vo)
- net VDD_A: now also J6.1 (Pin_1), R1.1
- net VSS_A: now reaches J3.1 (Pin_1), J4.2 (Pin_2), PS1.3 (-Vo)
- net VSS_A: now also D1.1 (K), J6.2 (Pin_2)
- net VDD_B: now reaches J3.2 (Pin_2), J5.1 (Pin_1), PS2.4 (+Vo)
- net VDD_B: now also J6.3 (Pin_3), R2.1
- net VSS_B: now reaches J5.2 (Pin_2), PS2.3 (-Vo)
- net VSS_B: now also D2.1 (K), J6.4 (Pin_4)
- new net: D2.2 (A), R2.2
- new net: D1.2 (A), R1.2
Other:
- moved on the sheet: H1, H2, H3, H4, J1, J2, J3, J4, PS1, PS2
